File: DCDC.kicad_sch (KiCad schematic)
At the start: 24 parts, among them U11 LM76005RNPR

Commit message: New conns for xESC
Added new connectors into the design for motors.
Changed lines of the file:
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@@
 (kicad_sch
-	(version 20231120)
+	(version 20250114)
 	(generator "eeschema")
-	(generator_version "8.0")
+	(generator_version "9.0")
 	(paper "A3")
 	(junction
@@
 	(label "BIAS"
 		(at 346.71 172.72 0)
-		(fields_autoplaced yes)
 		(effects
 			(font
@@
 	(label "BIAS"
 		(at 204.47 140.97 0)
-		(fields_autoplaced yes)
 		(effects
 			(font
@@
 		(shape input)
 		(at 72.39 128.27 180)
-		(fields_autoplaced yes)
 		(effects
 			(font
@@
 		(shape output)
 		(at 355.6 128.27 0)
-		(fields_autoplaced yes)
 		(effects
 			(font
