File: hw-openmower-universal.kicad_pcb (KiCad board)
At the start: 4 copper layers, 205 x 167.3 mm, 430 parts, among them J1 Conn_01x04, J10 Screw_Terminal_01x02, J12 xcore, J13 Screw_Terminal_01x02, J14 Conn_01x02, J15 Conn_01x04, J16 Conn_01x05, J17 Conn_01x02, J19 Conn_01x02, J2 Conn_02x04_Odd_Even, J22 Screw_Terminal_01x03, J23 Conn_01x05, J24 Conn_01x02, J27 Conn_01x05, J28 Conn_01x03_Male, J29 Conn_01x05, J3 Screw_Terminal_01x03, J30 Conn_01x03_Male, J31 Conn_01x03_Pin, J32 Conn_01x05_Pin, J33 10127820-0821LF, J34 Screw_Terminal_01x03, J35 Screw_Terminal_01x03, J36 Conn_02x03_Odd_Even, J37 Conn_02x03_Odd_Even, J38 Conn_02x03_Odd_Even, J4 Conn_02x05_Odd_Even, J45 RJ12, J46 10127820-0821LF, J47 10127820-0621GLF, J48 RJ45, J49 10127820-1022LF, J5 Conn_02x08_Odd_Even, J52 Conn_01x03_Male, J54 Conn_01x03_Male, J56 Screw_Terminal_01x02, J57 Conn_01x02, J58 Screw_Terminal_01x02, J59 Conn_01x02, J6 USB_A_Stacked, J60 Screw_Terminal_01x02, J61 Conn_01x02, J62 Screw_Terminal_01x02, J63 Conn_01x02, J7 HR911130A, J8 HR911130A, J9 Conn_01x02, M1 Fan, Q1 AO3400A, Q2 AO3400A, Q6 BSC0702LS, Q7 BSC0702LS, Q8 BSC0702LS, Q9 BSC0702LS, U10 xESC2, U11 LM76005RNPR, U12 AMS1117-3.3, U14 Fuse Holder, U15 Fuse Holder, U16 Fuse Holder, U17 Fuse Holder, U18 2.54mm 2x2 socket, U19 2.54mm 2x2 socket, U20 2.54mm 2x2 socket, U21 2.54mm 2x2 socket, U22 2.54mm 2x2 socket, U23 2.54mm 2x2 socket, U24 2.54mm 2x2 socket, U25 2.54mm 2x2 socket, U26 2.54mm 2x2 socket, U27 BQ25756RRVR, U28 LV2862XDDC, U29 LV2862XDDC, U3 TPS2065CDBV, U30 2.54mm 1x6 socket, U31 2.54mm 1x6 socket, U32 2.54mm 1x6 socket, U33 2.54mm 1x6 socket, U34 2.54mm 1x6 socket, U35 2.54mm 1x6 socket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

Commit message: Routing progress
Parts:
- removed R59: 2.2k, Resistor_SMD:R_0805_2012Metric
- added A1: Feather_ZED-F9P, Module:Adafruit_Feather_WithMountingHoles, F.Cu at (181.2, 170.2)
- added B1: MouseBite, Panelization:MouseBite-Slot_2.0x2.0mm_outset_D0.5mm_P0.85mm_3h, F.Cu at (10.8, -5.99)
- added R20: 1k, Resistor_SMD:R_0805_2012Metric, F.Cu at (182.3, 174.9)
- added R26: 150R, Resistor_SMD:R_0603_1608Metric, F.Cu at (174.6, 181.9)
Connections:
- C102 pad 1: /xESC_motor/5V -> /5V
- C103 pad 1: /xESC_motor/5V -> /5V
- C107 pad 1: /xESC2/5V -> /5V
- C108 pad 1: /xESC2/5V -> /5V
- C111 pad 1: /subpcb_logic/AGPIO4 -> /subpcb_charger/V_CHARGE_SENSE
- C21 pad 1: /xESC/5V -> /5V
- C35 pad 1: /xESC/5V -> /5V
- C37 pad 2: /5V -> /GPS/5V
- C63 pad 2: /5V -> /GPS/5V
- D23 pad 1: /subpcb_logic/AGPIO4 -> /subpcb_charger/V_CHARGE_SENSE
- D24 pad 1: /xESC_motor/5V -> /5V
- D25 pad 2: /5V -> /GPS/5V
- D28 pad 1: /xESC2/5V -> /5V
- D29 pad 2: /5V -> /subpcb_charger/5V
- D3 pad 2: /V_BATTERY -> /subpcb_charger/V_BATTERY
- D31 pad 2: /xESC/5V -> /5V
- D32 pad 2: /xESC_motor/5V -> /5V
- D33 pad 2: /xESC2/5V -> /5V
- D39 pad 2: /5V -> /subpcb_charger/5V
- D4 pad 1: /xESC/5V -> /5V
- D5 pad 2: /5V -> /subpcb_charger/5V
- D6 pad 2: /5V -> /subpcb_charger/5V
- F1 pad 2: /V_BATTERY -> /subpcb_charger/V_BATTERY
- J12 pad 77: /UART6.RX -> /subpcb_logic/UART6.RX
- J12 pad 92: /I2C1.SDA -> /subpcb_logic/I2C1.SDA
- J12 pad 94: /I2C1.SCL -> /subpcb_logic/I2C1.SCL
- J16 pad 2: /UART6.RX -> /subpcb_logic/UART6.RX
- J16 pad 3: /UART6.TX -> /subpcb_logic/UART6.TX
- J23 pad 2: /I2C1.SDA -> /subpcb_logic/I2C1.SDA
- J23 pad 3: /I2C1.SCL -> /subpcb_logic/I2C1.SCL
- J27 pad 1: /5V -> /subpcb_charger/5V
- J27 pad 2: /I2C1.SDA -> /subpcb_charger/I2C.SDA
- J27 pad 3: /I2C1.SCL -> /subpcb_charger/I2C.SCL
- J27 pad 4: /subpcb_logic/AGPIO4 -> /subpcb_charger/V_CHARGE_SENSE
- J29 pad 1: /5V -> /GPS/5V
- J29 pad 2: /UART6.RX -> /GPS/TXD
- J29 pad 3: /UART6.TX -> /GPS/RXD
- J36 pad 1: /xESC/5V -> /5V
- J37 pad 1: /xESC_motor/5V -> /5V
- J38 pad 1: /xESC2/5V -> /5V
- J56 pad 2: /V_BATTERY -> /subpcb_charger/V_BATTERY
- J57 pad 2: /V_BATTERY -> /subpcb_charger/V_BATTERY
- J58 pad 2: /V_BATTERY -> /subpcb_charger/V_BATTERY
- J59 pad 2: /V_BATTERY -> /subpcb_charger/V_BATTERY
- J60 pad 2: /V_BATTERY -> /subpcb_charger/V_BATTERY
- J61 pad 2: /V_BATTERY -> /subpcb_charger/V_BATTERY
- J62 pad 2: /V_BATTERY -> /subpcb_charger/V_BATTERY
- J63 pad 2: /V_BATTERY -> /subpcb_charger/V_BATTERY
- JP2 pad 1: /V_BATTERY -> /subpcb_charger/V_BATTERY
- L5 pad 2: /xESC/5V -> /5V
- L6 pad 2: /xESC_motor/5V -> /5V
- L7 pad 2: /xESC2/5V -> /5V
- R10 pad 1: /xESC/5V -> /5V
- R28 pad 1: /xESC_motor/5V -> /5V
- R31 pad 1: /xESC2/5V -> /5V
- R54 pad 1: /subpcb_logic/AGPIO4 -> /subpcb_charger/V_CHARGE_SENSE
- R55 pad 2: /subpcb_logic/AGPIO4 -> /subpcb_charger/V_CHARGE_SENSE
- R6 pad 1: /UART6.TX -> /subpcb_logic/UART6.TX
- U10 pad 5V: /xESC2/5V -> /5V
- U12 pad 3: /5V -> /GPS/5V
- U27 pad 1: /I2C1.SCL -> /subpcb_charger/I2C.SCL
- U27 pad 2: /I2C1.SDA -> /subpcb_charger/I2C.SDA
- U8 pad 5V: /xESC/5V -> /5V
- U9 pad 5V: /xESC_motor/5V -> /5V
- XA1 pad 5V1: /5V -> /GPS/5V
- XA1 pad D0: Net-(XA1-TXD) -> /GPS/TXD_R
- XA1 pad D1: /UART6.TX -> /GPS/RXD
Routing:
- net /I2C1.SDA: track 148.7 -> 0.00 mm, vias 3 -> 0
- net /I2C1.SCL: track 146.8 -> 0.00 mm, vias 4 -> 0
- net /xESC_motor/5V: track 127.4 -> 0.00 mm, vias 2 -> 0
- net /xESC2/5V: track 127.4 -> 0.00 mm, vias 2 -> 0
- net /xESC/5V: track 127.4 -> 0.00 mm, vias 2 -> 0
- net /GPS/RXD: track 0.00 -> 93.4 mm, vias 0 -> 1
- net /UART6.RX: track 79.8 -> 0.00 mm, vias 3 -> 0
- net /subpcb_charger/I2C.SDA: track 0.00 -> 79.5 mm, vias 0 -> 2
- net /subpcb_charger/I2C.SCL: track 0.00 -> 74.1 mm, vias 0 -> 1
- net /UART6.TX: track 73.3 -> 0.00 mm, vias 2 -> 0
- net /5V: track 122.5 -> 51.7 mm, vias 42 -> 36
- net /subpcb_logic/I2C1.SCL: track 0.00 -> 69.2 mm, vias 0 -> 1
- net /subpcb_logic/I2C1.SDA: track 0.00 -> 69.1 mm, vias 0 -> 1
- net /GPS/TXD_R: track 0.00 -> 59.2 mm
- net /GPS/TXD: track 0.00 -> 46.8 mm, vias 0 -> 1
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- added copper zone on F.Cu, net /xESC2/PHASE.U
- added copper zone on In2.Cu, net /xESC2/PHASE.V
- added copper zone on B.Cu, net /xESC2/PHASE.W
- added copper zone on B.Cu, net /xESC_motor/PHASE.U
- added copper zone on B.Cu, net /xESC_motor/PHASE.V
- added copper zone on In2.Cu, net /xESC_motor/PHASE.W
- removed copper zone on B.Cu, net /V_BATTERY
- removed copper zone on In1.Cu, net /V_BATTERY
- removed copper zone on In2.Cu, net GND
