File: hw-openmower-universal.kicad_pcb (KiCad board)
At the start: 4 copper layers, 205 x 167.3 mm, 404 parts, among them J1 Conn_01x04, J10 Screw_Terminal_01x02, J12 xcore, J13 Screw_Terminal_01x02, J14 Conn_01x02, J15 Conn_01x04, J16 Conn_01x05, J17 Conn_01x02, J19 Conn_01x02, J2 Conn_02x04_Odd_Even, J23 Conn_01x05, J24 Conn_01x02, J27 Conn_01x05, J29 Conn_01x05, J3 Screw_Terminal_01x03, J30 Conn_01x03_Male, J31 Conn_01x03_Pin, J32 Conn_01x05_Pin, J33 10127820-0821LF, J36 Conn_02x03_Odd_Even, J37 Conn_02x03_Odd_Even, J38 Conn_02x03_Odd_Even, J4 Conn_02x05_Odd_Even, J45 RJ12, J46 10127820-0821LF, J47 10127820-0621GLF, J48 RJ45, J49 10127820-1022LF, J5 Conn_02x08_Odd_Even, J54 Conn_01x03_Male, J56 Screw_Terminal_01x02, J57 Conn_01x02, J58 Screw_Terminal_01x02, J59 Conn_01x02, J60 Screw_Terminal_01x02, J61 Conn_01x02, J62 Screw_Terminal_01x02, J63 Conn_01x02, J7 HR911130A, J8 HR911130A, J9 Conn_01x02, M1 Fan, Q2 AO3400A, Q6 BSC0702LS, Q7 BSC0702LS, Q8 BSC0702LS, Q9 BSC0702LS, U10 xESC2, U11 LM76005RNPR, U12 AMS1117-3.3, U14 Fuse Holder, U15 Fuse Holder, U16 Fuse Holder, U17 Fuse Holder, U18 2.54mm 2x2 socket, U19 2.54mm 2x2 socket, U20 2.54mm 2x2 socket, U21 2.54mm 2x2 socket, U22 2.54mm 2x2 socket, U23 2.54mm 2x2 socket, U24 2.54mm 2x2 socket, U25 2.54mm 2x2 socket, U26 2.54mm 2x2 socket, U27 BQ25756RRVR, U28 LV2862XDDC, U29 LV2862XDDC, U3 TPS2065CDBV, U30 2.54mm 1x6 socket, U31 2.54mm 1x6 socket, U32 2.54mm 1x6 socket, U33 2.54mm 1x6 socket, U34 2.54mm 1x6 socket, U35 2.54mm 1x6 socket, U36 2.54mm 1x9 socket, U37 2.54mm 1x9 socket, U38 2.54mm 1x9 socket, U39 2.54mm 1x5 socket, U40 2.54mm 1x5 socket, U41 2.54mm 1x5 socket, U42 2.54mm 1x6 socket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

Commit message: Review ready layout
DRC mostly clean.  Need to add GND via stitching and GND return vias yet, and general review
Parts:
- removed D24, D28, D4: SS14, Diode_SMD:D_SMA
- added B2: MouseBite, Panelization:MouseBite-Slot_2.0x2.0mm_inset_D0.5mm_P0.85mm_4h_Trace, F.Cu at (235.5, 122.5)
- added B3: MouseBite, Panelization:MouseBite-Slot_2.0x2.0mm_inset_D0.5mm_P0.85mm_4h_Trace, F.Cu at (102.0, 122.5)
- added B4: MouseBite, Panelization:MouseBite-Slot_2.0x2.0mm_inset_D0.5mm_P0.85mm_4h_Trace, F.Cu at (203.5, 122.5)
- added B5: MouseBite, Panelization:MouseBite-Slot_2.0x2.0mm_inset_D0.5mm_P0.85mm_4h_Trace, F.Cu at (141.5, 122.5)
- added B6: MouseBite, Panelization:MouseBite-Slot_2.0x2.0mm_inset_D0.5mm_P0.85mm_4h_Trace, F.Cu at (164.5, 122.5)
- added B7: MouseBite, Panelization:MouseBite-Slot_2.0x2.0mm_inset_D0.5mm_P0.85mm_4h_Trace, F.Cu at (155.2, 135.8)
- added B8: MouseBite, Panelization:MouseBite-Slot_2.0x2.0mm_inset_D0.5mm_P0.85mm_4h_Trace, F.Cu at (155.2, 170.2)
- added B9: MouseBite, Panelization:MouseBite-Slot_2.0x2.0mm_inset_D0.5mm_P0.85mm_4h_Trace, F.Cu at (155.2, 153.5)
- B1: footprint Panelization:MouseBite-Slot_2.0x2.0mm_outset_D0.5mm_P0.85mm_3h -> Panelization:MouseBite-Slot_2.0x2.0mm_inset_D0.5mm_P0.85mm_4h_Trace
- moved B1 137.1 mm to (58.5, 122.5)
- moved H6 13.1 mm to (237.5, 176.5)
- moved H5 12.9 mm to (237.5, 128.8)
- moved C84 11.1 mm to (91.7, 146.0)
- moved kibuzzard-67111937 11.1 mm to (55.8, 167.2)
- moved C42 11.1 mm to (105.1, 173.1)
- moved C50 11.1 mm to (86.1, 165.9)
- moved C78 11.1 mm to (93.5, 148.8)
- moved D2 11.1 mm to (97.2, 151.3)
- moved D23 11.1 mm to (144.7, 158.8)
- moved H10 11.1 mm to (160.1, 176.8)
- moved H13 11.1 mm to (148.1, 128.8)
- moved H15 11.1 mm to (160.1, 128.8)
- moved H20 11.1 mm to (148.1, 176.8)
- moved H23 11.1 mm to (49.1, 128.8)
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Connections:
- C84 pad 1: Net-(U27-REGN) -> /subpcb_charger/Charger/REGN
- U27 pad 24: Net-(U27-REGN) -> /subpcb_charger/Charger/REGN
Routing:
- net /subpcb_logic/3.3V: track 20.6 -> 110.6 mm, vias 10 -> 11
- net /subpcb_charger/V_CHARGE_SENSE: track 2.90 -> 23.3 mm
- net /subpcb_charger/V_CHARGE: track 66.7 -> 85.1 mm
- net /subpcb_logic/Connectors/ETH1.PAIR_B_P: track 42.6 -> 57.8 mm, vias 0 -> 1
- net /subpcb_logic/Connectors/ETH1.PAIR_B_N: track 38.0 -> 48.2 mm, vias 0 -> 1
- net /5V: track 270.4 -> 260.5 mm, vias 47 -> 44
- net GND: track 281.2 -> 289.0 mm, vias 317 -> 314
- net /subpcb_logic/Connectors/ETH1.PAIR_D_N: track 34.6 -> 38.5 mm, vias 0 -> 1
- net Net-(D21-A): track 2.99 -> 6.55 mm
- net /subpcb_logic/Connectors/ETH1.PAIR_A_N: track 50.3 -> 53.7 mm
- net /subpcb_logic/Connectors/ETH1.PAIR_C_P: track 45.7 -> 49.1 mm
- net /subpcb_logic/UART8.RX: track 3.27 -> 0.00 mm, vias 1 -> 0
- net /subpcb_logic/AGPIO1: track 116.9 -> 113.9 mm
- net /subpcb_logic/Connectors/5V_SW: track 4.34 -> 6.49 mm, vias 0 -> 2
- net /subpcb_logic/Connectors/ETH1.PAIR_D_P: track 37.9 -> 38.1 mm, vias 0 -> 1
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- added copper zone on In2.Cu, net /GPS/5V
- added copper zone on F.Cu, net /V_BATTERY
- added copper zone on In2.Cu, net /subpcb_logic/Connectors/5V_SW
- added copper zone on In2.Cu, net GND
Other:
- board size 205 x 167.3 mm -> 198.7 x 156.3 mm
- board text removed: "${REFERENCE}"
