File: hw-openmower-universal.kicad_pcb (KiCad board)
At the start: 4 copper layers, 198.7 x 156.3 mm, 409 parts, among them J1 Conn_01x04, J10 Screw_Terminal_01x02, J12 xcore, J13 Screw_Terminal_01x02, J14 Conn_01x02, J15 Conn_01x04, J16 Conn_01x05, J17 Conn_01x02, J19 Conn_01x02, J2 Conn_02x04_Odd_Even, J23 Conn_01x05, J24 Conn_01x02, J27 Conn_01x05, J29 Conn_01x05, J3 Screw_Terminal_01x03, J30 Conn_01x03_Male, J31 Conn_01x03_Pin, J32 Conn_01x05_Pin, J33 10127820-0821LF, J36 Conn_02x03_Odd_Even, J37 Conn_02x03_Odd_Even, J38 Conn_02x03_Odd_Even, J4 Conn_02x05_Odd_Even, J45 RJ12, J46 10127820-0821LF, J47 10127820-0621GLF, J48 RJ45, J49 10127820-1022LF, J5 Conn_02x08_Odd_Even, J54 Conn_01x03_Male, J56 Screw_Terminal_01x02, J57 Conn_01x02, J58 Screw_Terminal_01x02, J59 Conn_01x02, J60 Screw_Terminal_01x02, J61 Conn_01x02, J62 Screw_Terminal_01x02, J63 Conn_01x02, J7 HR911130A, J8 HR911130A, J9 Conn_01x02, M1 Fan, Q2 AO3400A, Q6 BSC0702LS, Q7 BSC0702LS, Q8 BSC0702LS, Q9 BSC0702LS, U10 xESC2, U11 LM76005RNPR, U12 AMS1117-3.3, U14 Fuse Holder, U15 Fuse Holder, U16 Fuse Holder, U17 Fuse Holder, U18 2.54mm 2x2 socket, U19 2.54mm 2x2 socket, U20 2.54mm 2x2 socket, U21 2.54mm 2x2 socket, U22 2.54mm 2x2 socket, U23 2.54mm 2x2 socket, U24 2.54mm 2x2 socket, U25 2.54mm 2x2 socket, U26 2.54mm 2x2 socket, U27 BQ25756RRVR, U28 LV2862XDDC, U29 LV2862XDDC, U3 TPS2065CDBV, U30 2.54mm 1x6 socket, U31 2.54mm 1x6 socket, U32 2.54mm 1x6 socket, U33 2.54mm 1x6 socket, U34 2.54mm 1x6 socket, U35 2.54mm 1x6 socket, U36 2.54mm 1x9 socket, U37 2.54mm 1x9 socket, U38 2.54mm 1x9 socket, U39 2.54mm 1x5 socket, U40 2.54mm 1x5 socket, U41 2.54mm 1x5 socket, U42 2.54mm 1x6 socket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

Commit message: v1.0.0 - released to manufacturing
Released to manufacturing on 5/27/2026
Parts:
- C17, C18, C63: value 100nF -> 100nF@50V
- J50: value ~ -> KH-2AF1804ZJ-14.2JB
- moved LOGO2 36.4 mm to (234.7, 115.6)
- moved kibuzzard-67111FFB 2.54 mm to (134.7, 138.0), turned to 0 degrees
- moved kibuzzard-6711201C 1.61 mm to (149.2, 156.8), turned to 0 degrees
- moved kibuzzard-67111FDF 1.60 mm to (93.8, 138.2), turned to 0 degrees
- moved kibuzzard-6716385D 1.02 mm to (235.6, 31.2)
- moved kibuzzard-67111FCC 0.32 mm to (72.2, 137.9), turned to 0 degrees
- moved kibuzzard-67111FEA 0.14 mm to (112.2, 138.1), turned to 0 degrees
Routing:
- net /subpcb_logic/Connectors/ETH2.PAIR_B_N: track 19.6 -> 31.2 mm, vias 0 -> 1
- net /subpcb_logic/I2C4_ID.SDA: track 86.1 -> 96.9 mm
- net /subpcb_logic/I2C4_ID.SCL: track 89.0 -> 98.7 mm
- net /subpcb_logic/Connectors/ETH2.PAIR_B_P: track 21.6 -> 31.2 mm, vias 0 -> 1
- net /subpcb_logic/Connectors/ETH1.PAIR_B_P: track 57.8 -> 49.5 mm
- net GND: track 289.0 -> 297.3 mm, vias 314 -> 1370
- net /5V: track 260.5 -> 267.3 mm, vias 44 -> 45
- net Net-(J8-Pad14): track 32.3 -> 28.3 mm
- net /subpcb_logic/Connectors/USBH2.P: track 131.1 -> 134.9 mm
- net /subpcb_logic/Connectors/USBH2.N: track 131.7 -> 135.0 mm
- net /subpcb_logic/Connectors/ETH2.PAIR_A_N: track 27.5 -> 30.6 mm
- net /subpcb_logic/Connectors/ETH1.PAIR_C_P: track 49.1 -> 46.0 mm
- net /subpcb_logic/SPI2.MISO: track 91.3 -> 94.0 mm
- net Net-(Q9-G): track 24.6 -> 26.7 mm
- net /subpcb_logic/Connectors/ETH1.PAIR_A_P: track 53.9 -> 52.0 mm
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- added copper zone on In1.Cu, net /subpcb_logic/3.3V
- removed copper zone on In1.Cu, net /GPS/3.3V
- removed copper zone on In1.Cu, net /GPS/5V
Other:
- board text added: "OpenMower Mainboard for Husqvarna 115h v1.0.0 License CC BY 4.0 https://github.com/laberge1/hw-openmower-universal-husqvarna115h Forked from: https://github.com/ClemensElflein/OpenMower"
- board text removed: "OpenMower Universal Mainboard ${git_version} License CC BY 4.0 https://github.com/ClemensElflein/OpenMower"
