File: Connectors.kicad_sch (KiCad schematic)
At the start: 15 parts, among them J6 USB_A_Stacked, J7 HR911130A, J8 HR911130A, U3 TPS2065CDBV

Commit message: Routing progress and vertical USB
Parts:
- added J50: ~, USB:Kinghelm_USB_dual_vert, symbol USB:kinghelm_KH-2AF1804ZJ-14.2JB
Connections:
- net GND: now also J50.4 (GND), J50.8 (GND), J50.9 (SHLDGND)
- net USBH1.N: now also J50.2 (D-)
- net USBH1.P: now also J50.3 (D+)
- net USBH2.N: now also J50.6 (D-)
- net USBH2.P: now also J50.7 (D+)
- net 5V_SW: now reaches C5.1, C9.1, J6.1 (VBUS1), J6.5 (VBUS2), U3.1 (OUT)
- net 5V_SW: now also J50.1 (VCC), J50.5 (VCC)

Commit message: Further routing progress
Parts:
- removed J6: USB_A_Stacked, Connector_USB:USB_A_Wuerth_61400826021_Horizontal_Stacked, symbol Connector:USB_A_Stacked
Connections:
- net 5V_SW: now also R8.2, U3.3 (~{FLT}); no longer C5.1, C9.1, U3.1 (OUT)
- new net: C5.1, C9.1, U3.1 (OUT)
Other:
- moved on the sheet: J50
